File: bearer/pi485carrier.kicad_pcb (KiCad board)
At the start: 2 copper layers, 62 x 30 mm, 21 parts, among them P1 PWR, P2 Rasperry Pi, P3 Latch Disable, P4 TERM, P5 CONN_01X04, P6 CONN_01X04, Q1 2N4401, Q2 2N4401, Q3 2N4401, U1 NE555

Commit message: Renaming carrier to bearer...
Other:
- board text added: "Pi485 Bearer Rev 1.1.0"
- board text removed: "Pi485 Carrier Rev 1.1.0"
Changed lines of the file:
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@@
     (descr "TO-92 leads in-line, wide, drill 0.8mm (see NXP sot054_po.pdf)")
     (tags "to-92 sc-43 sc-43a sot54 PA33 transistor")
-    (fp_text reference Q3 (at 4.7 -2.965 360) (layer F.SilkS)
+    (fp_text reference Q3 (at 4.7 -2.965) (layer F.SilkS)
       (effects (font (size 1 1) (thickness 0.15)))
     )
@@
     (arrow2b (pts (xy 37.465 17.955) (xy 38.591504 17.368579)))
   )
-  (gr_text "Pi485 Carrier\nRev 1.1.0" (at 88.265 48.26) (layer F.SilkS)
+  (gr_text "Pi485 Bearer\nRev 1.1.0" (at 88.265 48.26) (layer F.SilkS)
     (effects (font (size 1.5 1.5) (thickness 0.3)))
   )
