File: standalone/pi485.sch (KiCad schematic (older format))
At the start: 29 parts, among them J1 RS485, P1 Rasperry Pi, P2 PWR, P3 TERM, P4 RO, Q1 2N3904, Q2 2N3904, Q3 2N3904, Q4 2N3906, U1 NE555, U2 MAX485

Commit message: 1.1.1 schematics, trace plots, etc.
Parts:
- added C4: 10nF, Capacitors_THT:C_Rect_L4_W2.5_P2.5, symbol C
- added R12: 10k, Resistors_THT:Resistor_Horizontal_RM10mm, symbol R
Connections:
- net GND: now also C4.2, R12.1
- net at U1.3 (Q), U2.2 (~RE), U2.3 (DE): now also R12.2
- net at P4.2 (P2), U1.5 (CV): now also C4.1
Other:
- moved on the sheet: P4
Changed lines of the file:
@@
 Sheet 1 1
 Title "Pi485"
-Date "2017-02-12"
-Rev "1.1.0"
+Date "2017-02-20"
+Rev "1.1.1"
 Comp "Bryan Varner"
 Comment1 ""
@@
 L CONN_01X02 P4
 U 1 1 587D51D9
-P 4800 6400
-F 0 "P4" H 4800 6550 50  0000 C CNN
-F 1 "RO" V 4900 6400 50  0000 C CNN
-F 2 "Pin_Headers:Pin_Header_Straight_1x02" H 5450 6650 50  0001 C CNN
-F 3 "" H 4800 6400 50  0000 C CNN
-	1    4800 6400
+P 4650 6500
+F 0 "P4" H 4650 6650 50  0000 C CNN
+F 1 "RO" V 4750 6500 50  0000 C CNN
+F 2 "Pin_Headers:Pin_Header_Straight_1x02" H 5300 6750 50  0001 C CNN
+F 3 "" H 4650 6500 50  0000 C CNN
+	1    4650 6500
 	-1   0    0    1
 $EndComp
@@
 Connection ~ 6400 5850
 Wire Wire Line
-	5000 6450 6000 6450
+	5150 6450 6000 6450
 Connection ~ 5500 6450
 Wire Wire Line
@@
 	8000 2600 8000 2700
 Wire Wire Line
-	7100 6000 7100 3200
+	7100 3200 7100 5950
 Wire Wire Line
 	7500 2650 7500 2300
@@
 Connection ~ 6400 6050
 Wire Wire Line
-	5000 6350 5000 5850
+	4850 5850 5000 5850
 Wire Wire Line
 	7400 4550 7400 4750
@@
 	6400 6450 6300 6450
 Wire Wire Line
-	4300 6750 6800 6750
+	4300 6750 6650 6750
 Connection ~ 5500 6750
 Wire Wire Line
@@
 	2850 6400 4300 6400
 Wire Wire Line
-	6800 6750 6800 6000
+	6650 6750 6650 5950
 Wire Wire Line
 	5150 2800 5150 3300
@@
 Connection ~ 7400 5550
 Wire Wire Line
-	6800 6000 7100 6000
+	6650 5950 7100 5950
 Wire Wire Line
 	7800 5200 7800 5550
+$Comp
+L C C4
+U 1 1 58AB7251
+P 5000 6450
+F 0 "C4" V 5100 6600 50  0000 C CNN
+F 1 "10nF" V 5100 6300 50  0000 C CNN
+F 2 "Capacitors_THT:C_Rect_L4_W2.5_P2.5" V 5200 6150 50  0001 C CNN
+F 3 "" H 5000 6450 50  0000 C CNN
+	1    5000 6450
+	0    -1   -1   0
+$EndComp
+Wire Wire Line
+	4850 5850 4850 6450
+Wire Wire Line
+	4850 6550 4850 6750
+Connection ~ 4850 6750
+$Comp
+L R R12
+U 1 1 58AB7CF0
+P 6650 5800
+F 0 "R12" V 6730 5800 50  0000 C CNN
+F 1 "10k" V 6650 5800 50  0000 C CNN
+F 2 "Resistors_THT:Resistor_Horizontal_RM10mm" H 5750 5800 50  0001 C CNN
+F 3 "" H 6650 5800 50  0000 C CNN
+	1    6650 5800
+	-1   0    0    1
+$EndComp
 $EndSCHEMATC

Commit message: Updates for jumpered biasing on standalone boards. The silly bearer modules you can just unsolder the biasing resistors if it becomes an issue. I should probably add jumpering for that too, but at this point, I just don't much care. A slight modification to those silly SMT boards really isn't that hard...
Parts:
- P3: value TERM -> TERM / BIAS; footprint Pin_Headers:Pin_Header_Straight_1x02 -> Pin_Headers:Pin_Header_Straight_2x03; symbol CONN_01X02 -> CONN_02X03
- R1, R12, R4, R6: footprint Resistors_THT:Resistor_Horizontal_RM10mm -> Resistors_THT:Resistor_Horizontal_RM7mm
Connections:
- net at J1.1, U2.6 (A): now also P3.3 (P3), P3.5 (P5); no longer P3.2 (P2), R6.1
- net at J1.2, R5.1, U2.7 (B): now also P3.4 (P4); no longer R4.2
- net at R5.2: now also P3.6 (P6); no longer P3.1 (P1)
- new net: P3.2 (P2), R4.2
- new net: P3.1 (P1), R6.1
Other:
- moved on the sheet: R4, R5, R6
Changed lines of the file:
@@
 Sheet 1 1
 Title "Pi485"
-Date "2017-02-20"
+Date "2017-02-21"
 Rev "1.1.1"
 Comp "Bryan Varner"
@@
 F 0 "R1" H 7480 4900 50  0000 C CNN
 F 1 "200" V 7400 4900 50  0000 C CNN
-F 2 "Resistors_THT:Resistor_Horizontal_RM10mm" V 7550 4200 50  0001 C CNN
+F 2 "Resistors_THT:Resistor_Horizontal_RM7mm" V 7550 4200 50  0001 C CNN
 F 3 "" H 7400 4900 50  0000 C CNN
 	1    7400 4900
@@
 L R R5
 U 1 1 586EB6FC
-P 8000 2450
-F 0 "R5" V 8080 2450 50  0000 C CNN
-F 1 "120" V 8000 2450 50  0000 C CNN
-F 2 "Resistors_THT:Resistor_Horizontal_RM10mm" H 8850 2650 50  0001 C CNN
-F 3 "" H 8000 2450 50  0000 C CNN
-	1    8000 2450
+P 8000 2000
+F 0 "R5" V 8080 2000 50  0000 C CNN
+F 1 "120" V 8000 2000 50  0000 C CNN
+F 2 "Resistors_THT:Resistor_Horizontal_RM10mm" H 8850 2200 50  0001 C CNN
+F 3 "" H 8000 2000 50  0000 C CNN
+	1    8000 2000
 	1    0    0    -1
 $EndComp
@@
 L R R4
 U 1 1 586EB760
-P 8000 2050
-F 0 "R4" V 8080 2050 50  0000 C CNN
-F 1 "20k" V 8000 2050 50  0000 C CNN
-F 2 "Resistors_THT:Resistor_Horizontal_RM10mm" H 8850 2300 50  0001 C CNN
-F 3 "" H 8000 2050 50  0000 C CNN
-	1    8000 2050
+P 8200 2250
+F 0 "R4" V 8280 2250 50  0000 C CNN
+F 1 "20k" V 8200 2250 50  0000 C CNN
+F 2 "Resistors_THT:Resistor_Horizontal_RM7mm" H 9050 2500 50  0001 C CNN
+F 3 "" H 8200 2250 50  0000 C CNN
+	1    8200 2250
 	1    0    0    -1
 $EndComp
@@
 L R R6
 U 1 1 586EB7D4
-P 8000 3150
-F 0 "R6" V 8080 3150 50  0000 C CNN
-F 1 "20k" V 8000 3150 50  0000 C CNN
-F 2 "Resistors_THT:Resistor_Horizontal_RM10mm" H 8850 3300 50  0001 C CNN
-F 3 "" H 8000 3150 50  0000 C CNN
-	1    8000 3150
+P 8200 3050
+F 0 "R6" V 8280 3050 50  0000 C CNN
+F 1 "20k" V 8200 3050 50  0000 C CNN
+F 2 "Resistors_THT:Resistor_Horizontal_RM7mm" H 9050 3200 50  0001 C CNN
+F 3 "" H 8200 3050 50  0000 C CNN
+	1    8200 3050
 	1    0    0    -1
 $EndComp
@@
 (TXDO)_GPIO14
 $Comp
-L CONN_01X02 P3
+L CONN_02X03 P3
 U 1 1 586EFE3A
-P 8200 2750
-F 0 "P3" H 8200 2900 50  0000 C CNN
-F 1 "TERM" V 8300 2750 50  0000 C CNN
-F 2 "Pin_Headers:Pin_Header_Straight_1x02" H 8850 3000 50  0001 C CNN
-F 3 "" H 8200 2750 50  0000 C CNN
-	1    8200 2750
-	1    0    0    -1
+P 8100 2650
+F 0 "P3" H 8100 2800 50  0000 C CNN
+F 1 "TERM / BIAS" V 8100 2650 50  0000 C CNN
+F 2 "Pin_Headers:Pin_Header_Straight_2x03" H 8750 2900 50  0001 C CNN
+F 3 "" H 8100 2650 50  0000 C CNN
+	1    8100 2650
+	0    1    -1   0
 $EndComp
 Text Label 2500 2150 3    60   ~ 0
@@
 L VCC #PWR06
 U 1 1 586F01EA
-P 8250 3300
-F 0 "#PWR06" H 8250 3150 50  0001 C CNN
-F 1 "VCC" H 8250 3450 50  0000 C CNN
-F 2 "" H 8250 3300 50  0000 C CNN
-F 3 "" H 8250 3300 50  0000 C CNN
-	1    8250 3300
+P 8400 3200
+F 0 "#PWR06" H 8400 3050 50  0001 C CNN
+F 1 "VCC" H 8400 3350 50  0000 C CNN
+F 2 "" H 8400 3200 50  0000 C CNN
+F 3 "" H 8400 3200 50  0000 C CNN
+	1    8400 3200
 	1    0    0    -1
 $EndComp
@@
 L GND #PWR07
 U 1 1 586F0172
-P 8250 1900
-F 0 "#PWR07" H 8250 1650 50  0001 C CNN
-F 1 "GND" H 8250 1750 50  0000 C CNN
-F 2 "" H 8250 1900 50  0000 C CNN
-F 3 "" H 8250 1900 50  0000 C CNN
-	1    8250 1900
+P 8450 2100
+F 0 "#PWR07" H 8450 1850 50  0001 C CNN
+F 1 "GND" H 8450 1950 50  0000 C CNN
+F 2 "" H 8450 2100 50  0000 C CNN
+F 3 "" H 8450 2100 50  0000 C CNN
+	1    8450 2100
 	1    0    0    -1
 $EndComp
@@
 	6650 5650 6000 5650
 Connection ~ 6650 2900
-Connection ~ 8000 2300
-Connection ~ 8000 2900
-Wire Wire Line
-	8000 2300 8000 2200
-Wire Wire Line
-	8000 2800 8000 3000
+Connection ~ 8000 1850
+Connection ~ 8000 3500
+Wire Wire Line
+	8100 1850 8100 2400
+Wire Wire Line
+	8000 2900 8000 3500
 Wire Wire Line
 	2800 3000 6450 3000
@@
 	6550 3000 6700 3000
 Wire Wire Line
-	8000 3300 8250 3300
-Wire Wire Line
-	8250 1900 8000 1900
-Wire Wire Line
-	8000 2600 8000 2700
+	8200 3200 8400 3200
+Wire Wire Line
+	8450 2100 8200 2100
 Wire Wire Line
 	7100 3200 7100 5950
 Wire Wire Line
-	7500 2650 7500 2300
-Wire Wire Line
-	7500 2300 9000 2300
-Wire Wire Line
-	9000 2300 9000 2500
-Wire Wire Line
-	7500 2850 7500 2900
-Wire Wire Line
-	7500 2900 9000 2900
-Wire Wire Line
-	9000 2900 9000 2700
+	7500 2650 7500 1850
+Wire Wire Line
+	7500 1850 9000 1850
+Wire Wire Line
+	9000 1850 9000 2500
+Wire Wire Line
+	7500 2850 7500 3500
+Wire Wire Line
+	7500 3500 9000 3500
+Wire Wire Line
+	9000 3500 9000 2700
 Connection ~ 2500 2800
 Connection ~ 2600 2900
@@
 F 0 "R12" V 6730 5800 50  0000 C CNN
 F 1 "10k" V 6650 5800 50  0000 C CNN
-F 2 "Resistors_THT:Resistor_Horizontal_RM10mm" H 5750 5800 50  0001 C CNN
+F 2 "Resistors_THT:Resistor_Horizontal_RM7mm" H 5750 5800 50  0001 C CNN
 F 3 "" H 6650 5800 50  0000 C CNN
 	1    6650 5800
 	-1   0    0    1
 $EndComp
+Wire Wire Line
+	8000 2400 8000 2150
+Wire Wire Line
+	8100 2900 8100 3500
+Connection ~ 8100 3500
+Connection ~ 8100 1850
 $EndSCHEMATC
